File: A_Micromouse_Team_PCB_Rev1/_autosave-A_Micromouse_Team_PCB_Rev1.kicad_pcb (KiCad board)
At the start: 2 copper layers, 9 parts, among them J1 Conn_01x07_Pin, J2 Conn_01x07_Pin, J3 Conn_01x07_Pin, J5 Conn_01x06_Pin, J6 Conn_01x06_Pin, J8 Conn_01x07_Pin, U1 Teensy4.0, U2 BNO055, U3 TB6612FNG

Commit message: changed Net Classes
Parts:
- added J10: Conn_01x06, Connector_PinHeader_2.00mm:PinHeader_1x06_P2.00mm_Vertical, F.Cu at (74.1, 36.1)
- added J4: Conn_01x07_Pin, Connector_PinHeader_2.54mm:PinHeader_1x07_P2.54mm_Vertical, F.Cu at (50.4, 55.4)
- added J7: Conn_01x04_Socket, Connector_PinHeader_2.00mm:PinHeader_1x04_P2.00mm_Vertical, F.Cu at (68.6, 65.1)
- added J9: Conn_01x02_Socket, Connector_PinHeader_2.00mm:PinHeader_1x02_P2.00mm_Vertical, F.Cu at (72.6, 65.1)
- moved U1 24.7 mm to (111.8, 58.4)
- moved J3 23.6 mm to (45.7, 55.4)
- moved J1 23.6 mm to (36.4, 55.4)
- moved J2 23.6 mm to (41.1, 55.4)
- moved J5 19.8 mm to (59.7, 55.4)
- moved J6 19.8 mm to (64.3, 55.4)
- moved J8 19.8 mm to (55.0, 55.4)
- moved U3 18.6 mm to (71.8, 58.1)
- moved U2 10.9 mm to (60.9, 73.1)
Connections:
- J1 pad 6: unconnected-(J1-Pin_6-Pad6) -> Net-(J1-Pin_6)
- J2 pad 6: unconnected-(J2-Pin_6-Pad6) -> Net-(J2-Pin_6)
- J3 pad 6: unconnected-(J3-Pin_6-Pad6) -> Net-(J3-Pin_6)
- J5 pad 2: unconnected-(J5-Pin_2-Pad2) -> Net-(J5-Pin_2)
- J5 pad 3: unconnected-(J5-Pin_3-Pad3) -> Net-(J5-Pin_3)
- J6 pad 2: unconnected-(J6-Pin_2-Pad2) -> Net-(J6-Pin_2)
- J6 pad 3: unconnected-(J6-Pin_3-Pad3) -> Net-(J6-Pin_3)
- J8 pad 6: unconnected-(J8-Pin_6-Pad6) -> Net-(J8-Pin_6)
- U1 pad 10: unconnected-(U1-8_TX2_IN1-Pad10) -> Net-(U1-8_TX2_IN1)
- U1 pad 11: unconnected-(U1-9_OUT1C-Pad11) -> Net-(J6-Pin_2)
- U1 pad 12: unconnected-(U1-10_CS_MQSR-Pad12) -> Net-(J6-Pin_3)
- U1 pad 13: unconnected-(U1-11_MOSI_CTX1-Pad13) -> Net-(J5-Pin_2)
- U1 pad 14: unconnected-(U1-12_MISO_MQSL-Pad14) -> Net-(J5-Pin_3)
- U1 pad 20: unconnected-(U1-13_SCK_CRX1_LED-Pad20) -> Net-(U1-13_SCK_CRX1_LED)
- U1 pad 22: unconnected-(U1-15_A1_RX3_SPDIF_IN-Pad22) -> Net-(J7-Pin_2)
- U1 pad 23: unconnected-(U1-16_A2_RX4_SCL1-Pad23) -> Net-(U1-16_A2_RX4_SCL1)
- U1 pad 24: unconnected-(U1-17_A3_TX4_SDA1-Pad24) -> Net-(U1-17_A3_TX4_SDA1)
- U1 pad 29: unconnected-(U1-22_A8_CTX1-Pad29) -> Net-(U1-22_A8_CTX1)
- U1 pad 30: unconnected-(U1-23_A9_CRX1_MCLK1-Pad30) -> Net-(U1-23_A9_CRX1_MCLK1)
- U1 pad 4: unconnected-(U1-2_OUT2-Pad4) -> Net-(J4-Pin_6)
- U1 pad 5: unconnected-(U1-3_LRCLK2-Pad5) -> Net-(J3-Pin_6)
- U1 pad 6: unconnected-(U1-4_BCLK2-Pad6) -> Net-(J2-Pin_6)
- U1 pad 7: unconnected-(U1-5_IN2-Pad7) -> Net-(J1-Pin_6)
- U1 pad 8: unconnected-(U1-6_OUT1D-Pad8) -> Net-(J8-Pin_6)
- U1 pad 9: unconnected-(U1-7_RX2_OUT1A-Pad9) -> Net-(U1-7_RX2_OUT1A)
- U3 pad 15: unconnected-(U3-PWMB-Pad15) -> Net-(U1-7_RX2_OUT1A)
- U3 pad 16: unconnected-(U3-BIN2-Pad16) -> Net-(U1-23_A9_CRX1_MCLK1)
- U3 pad 17: unconnected-(U3-BIN1-Pad17) -> Net-(U1-22_A8_CTX1)
- U3 pad 18: unconnected-(U3-GND-Pad18) -> GND
- U3 pad 19: unconnected-(U3-STBY-Pad19) -> Net-(U1-13_SCK_CRX1_LED)
- U3 pad 20: unconnected-(U3-VCC-Pad20) -> +5V
- U3 pad 21: unconnected-(U3-AIN1-Pad21) -> Net-(U1-16_A2_RX4_SCL1)
- U3 pad 22: unconnected-(U3-AIN2-Pad22) -> Net-(U1-17_A3_TX4_SDA1)
- U3 pad 23: unconnected-(U3-PWMA-Pad23) -> Net-(U1-8_TX2_IN1)
- U3 pad 24: unconnected-(U3-VM1-Pad24) -> +12V
