File: A_Micromouse_Team_PCB_Rev1/A_Micromouse_Team_PCB_Rev1.kicad_sch (KiCad schematic)
At the start: 18 parts, among them J1 TOF2, J10 5V->12V, J2 TOF3, J3 TOF4, J4 TOF5, J5 Motor1, J6 Motor2, J7 NeoPixel, J8 TOF1, J9 Battery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

Commit message: finished revamped schematic
Connections:
- net SCL: now also U2.19 (COM1)
- net SDA: now also U2.20 (COM0)
- net at J7.2 (Pin_2): now also U1.29 (22_A8_CTX1)
Other:
- moved on the sheet: U2
Changed lines of the file:
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@@
   (no_connect (at 167.64 62.23))
   (no_connect (at 167.64 54.61))
-  (no_connect (at 71.12 148.59))
+  (no_connect (at 194.31 140.97))
   (no_connect (at 167.64 59.69))
   (no_connect (at 167.64 85.09))
@@
     (stroke (width 0) (type default))
   )
+  (wire (pts (xy 187.96 120.65) (xy 187.96 123.19))
+    (stroke (width 0) (type default))
+  )
   (wire (pts (xy 90.17 119.38) (xy 90.17 90.17))
     (stroke (width 0) (type default))
@@
   )
   (wire (pts (xy 68.58 43.18) (xy 93.98 43.18))
+    (stroke (width 0) (type default))
+  )
+  (wire (pts (xy 167.64 123.19) (xy 167.64 170.18))
     (stroke (width 0) (type default))
   )
@@
     )
   )
+  (global_label "SCL" (shape input) (at 175.26 148.59 180) (fields_autoplaced)
+    (effects (font (size 1.27 1.27)) (justify right))
+    (property "Intersheetrefs" "${INTERSHEET_REFS}" (at 168.7672 148.59 0)
+      (effects (font (size 1.27 1.27)) (justify right) hide)
+    )
+  )
   (global_label "SW4" (shape input) (at 116.84 129.54 0) (fields_autoplaced)
     (effects (font (size 1.27 1.27)) (justify left))
     (property "Intersheetrefs" "${INTERSHEET_REFS}" (at 123.6956 129.54 0)
       (effects (font (size 1.27 1.27)) (justify left) hide)
+    )
+  )
+  (global_label "SDA" (shape input) (at 175.26 146.05 180) (fields_autoplaced)
+    (effects (font (size 1.27 1.27)) (justify right))
+    (property "Intersheetrefs" "${INTERSHEET_REFS}" (at 168.7067 146.05 0)
+      (effects (font (size 1.27 1.27)) (justify right) hide)
     )
   )
@@
     )
   )
-  (symbol (lib_id "Sensor_Motion:BNO055") (at 67.31 148.59 0) (unit 1)
-    (in_bom yes) (on_board yes) (dnp no) (fields_autoplaced)
-    (property "Reference" "U2" (at 72.0441 128.27 0)
-      (effects (font (size 1.27 1.27)) (justify left))
-    )
-    (property "Value" "IMU" (at 72.0441 130.81 0)
-      (effects (font (size 1.27 1.27)) (justify left))
-    )
-    (property "Footprint" "MicromouseLibaryNew:MODULE_4754" (at 73.66 165.1 0)
+  (symbol (lib_id "Sensor_Motion:BNO055") (at 190.5 140.97 0) (unit 1)
+    (in_bom yes) (on_board yes) (dnp no) (fields_autoplaced)
+    (property "Reference" "U2" (at 195.2341 120.65 0)
+      (effects (font (size 1.27 1.27)) (justify left))
+    )
+    (property "Value" "IMU" (at 195.2341 123.19 0)
+      (effects (font (size 1.27 1.27)) (justify left))
+    )
+    (property "Footprint" "MicromouseLibaryNew:MODULE_4754" (at 196.85 157.48 0)
       (effects (font (size 1.27 1.27)) (justify left) hide)
     )
-    (property "Datasheet" "https://www.bosch-sensortec.com/media/boschsensortec/downloads/datasheets/bst-bno055-ds000.pdf" (at 67.31 143.51 0)
+    (property "Datasheet" "https://www.bosch-sensortec.com/media/boschsensortec/downloads/datasheets/bst-bno055-ds000.pdf" (at 190.5 135.89 0)
       (effects (font (size 1.27 1.27)) hide)
     )
@@
     )
   )
+  (symbol (lib_id "power:+5V") (at 187.96 120.65 0) (unit 1)
+    (in_bom yes) (on_board yes) (dnp no) (fields_autoplaced)
+    (property "Reference" "#PWR06" (at 187.96 124.46 0)
+      (effects (font (size 1.27 1.27)) hide)
+    )
+    (property "Value" "+5V" (at 187.96 115.57 0)
+      (effects (font (size 1.27 1.27)))
+    )
+    (property "Footprint" "" (at 187.96 120.65 0)
+      (effects (font (size 1.27 1.27)) hide)
+    )
+    (property "Datasheet" "" (at 187.96 120.65 0)
+      (effects (font (size 1.27 1.27)) hide)
+    )
+    (pin "1")
+    (instances
+      (project "A_Micromouse_Team_PCB_Rev1"
+        (path "/c13bd0ff-2c2c-4c0d-a2fb-bf65e79fa3e5"
+          (reference "#PWR06") (unit 1)
+        )
+      )
+    )
+  )
   (symbol (lib_id "power:+5V") (at 190.5 27.94 90) (unit 1)
     (in_bom yes) (on_board yes) (dnp no)
@@
     )
   )
-  (symbol (lib_id "power:+5V") (at 64.77 130.81 0) (unit 1)
-    (in_bom yes) (on_board yes) (dnp no) (fields_autoplaced)
-    (property "Reference" "#PWR06" (at 64.77 134.62 0)
-      (effects (font (size 1.27 1.27)) hide)
-    )
-    (property "Value" "+5V" (at 64.77 125.73 0)
-      (effects (font (size 1.27 1.27)))
-    )
-    (property "Footprint" "" (at 64.77 130.81 0)
-      (effects (font (size 1.27 1.27)) hide)
-    )
-    (property "Datasheet" "" (at 64.77 130.81 0)
-      (effects (font (size 1.27 1.27)) hide)
-    )
-    (pin "1")
-    (instances
-      (project "A_Micromouse_Team_PCB_Rev1"
-        (path "/c13bd0ff-2c2c-4c0d-a2fb-bf65e79fa3e5"
-          (reference "#PWR06") (unit 1)
-        )
-      )
-    )
-  )
   (symbol (lib_id "power:GND") (at 187.96 25.4 270) (unit 1)
     (in_bom yes) (on_board yes) (dnp no)
@@
     )
   )
-  (symbol (lib_id "power:GND") (at 64.77 166.37 0) (unit 1)
-    (in_bom yes) (on_board yes) (dnp no) (fields_autoplaced)
-    (property "Reference" "#PWR029" (at 64.77 172.72 0)
-      (effects (font (size 1.27 1.27)) hide)
-    )
-    (property "Value" "GND" (at 64.77 171.45 0)
-      (effects (font (size 1.27 1.27)))
-    )
-    (property "Footprint" "" (at 64.77 166.37 0)
-      (effects (font (size 1.27 1.27)) hide)
-    )
-    (property "Datasheet" "" (at 64.77 166.37 0)
-      (effects (font (size 1.27 1.27)) hide)
-    )
+  (symbol (lib_id "power:GND") (at 187.96 158.75 0) (unit 1)
+    (in_bom yes) (on_board yes) (dnp no) (fields_autoplaced)
+    (property "Reference" "#PWR029" (at 187.96 165.1 0)
+      (effects (font (size 1.27 1.27)) hide)
+    )
+    (property "Value" "GND" (at 187.96 163.83 0)
+      (effects (font (size 1.27 1.27)))
+    )
+    (property "Footprint" "" (at 187.96 158.75 0)
+      (effects (font (size 1.27 1.27)) hide)
+    )
+    (property "Datasheet" "" (at 187.96 158.75 0)
+      (effects (font (size 1.27 1.27)) hide)
+    )

Commit message: revamped schematic
Other:
- note added: "Please give this a read Edward"
Changed lines of the file:
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@@
     (stroke (width 0) (type default))
+  )
+  (text "Please give this a read Edward\n" (at 20.32 24.13 0)
+    (effects (font (size 1.27 1.27)) (justify left bottom))
   )
   (global_label "TOF2" (shape input) (at 111.76 67.31 180) (fields_autoplaced)

Commit message: checked all footprints and created a max footprint
Parts:
- added C1, C2, C3: C, Capacitor_THT:CP_Radial_D8.0mm_P2.50mm, symbol Device:C
- added J11, J12: MotorCageMount, MicromouseLibaryNew:motorMount, symbol Connector_Generic:Conn_01x01
- R1, R2, R3, R4: footprint (none) -> Resistor_THT:R_Axial_DIN0309_L9.0mm_D3.2mm_P12.70mm_Horizontal
Connections:
- net +3.3V: now also C3.2
- net GND: now also C1.2, C2.1, C3.1
- net at J9.1 (Pin_1), SW1.1: now also C1.1
- net at J10.1 (Pin_1), SW1.2: now also C2.2
Other:
- moved on the sheet: J1, J2, J3, J4, J8, U2
