File: A_Micromouse_Team_PCB_Rev1/_autosave-A_Micromouse_Team_PCB_Rev1.kicad_sch (KiCad schematic)
At the start: 23 parts, among them J1 TOF2, J10 5V->12V, J11 MotorCageMount, J12 MotorCageMount, J2 TOF3, J3 TOF4, J4 TOF5, J5 Motor1, J6 Motor2, J7 NeoPixel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

Commit message: Add files via upload
Parts:
- removed C1, C2, C3: C, Capacitor_THT:CP_Radial_D8.0mm_P2.50mm, symbol Device:C
- added J13: Battery, Connector_PinHeader_2.00mm:PinHeader_1x02_P2.00mm_Vertical, symbol Connector:Conn_01x02_Socket
- added R5, R6: R_US, Resistor_THT:R_Axial_DIN0309_L9.0mm_D3.2mm_P12.70mm_Horizontal, symbol Device:R_US
Connections:
- net +12V: now also U3.24 (VM1)
- net +3.3V: now also R5.2, R6.2
- net +5V: no longer J10.4 (Pin_4)
- net GND: now also J13.2 (Pin_2)
- net SCL: now also R6.1
- net SDA: now also R5.1
- net +5VD: now reaches J10.5 (Pin_5)
- net +5VD: now also J10.4 (Pin_4), J13.1 (Pin_1)
